File: pcb/df_selector.kicad_pcb (KiCad board)
At the start: 2 copper layers, 52.5 x 58.8 mm, 10 parts

Commit message: added stacked pcb
Routing:
- net (no net): track 578.9 -> 564.2 mm
- removed copper zone on B.Cu, net (none)
Changed lines of the file:
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@@
   (general
     (thickness 1.6)
-    (drawings 26)
-    (tracks 145)
+    (drawings 28)
+    (tracks 135)
     (zones 0)
     (modules 10)
@@
   )
   (setup
-    (last_trace_width 2)
+    (last_trace_width 0.25)
     (user_trace_width 0.5)
     (user_trace_width 1)
@@
   (module "4-channel logic level converter" (layer F.Cu)
     (at 0 0)
-    (fp_text reference REF** (at 0 0.5) (layer F.SilkS)
+    (fp_text reference REF** (at 55.8 38.9) (layer F.SilkS)
       (effects (font (size 1 1) (thickness 0.15)))
     )
@@
       (rotate (xyz 0 0 0))
     )
+  )
+  (dimension 58.75 (width 0.15) (layer Dwgs.User)
+    (gr_text "58.750 mm" (at 127.6 89.875 270) (layer Dwgs.User)
+      (effects (font (size 1 1) (thickness 0.15)))
+    )
+    (feature1 (pts (xy 124.5 119.25) (xy 126.886421 119.25)))
+    (feature2 (pts (xy 124.5 60.5) (xy 126.886421 60.5)))
+    (crossbar (pts (xy 126.3 60.5) (xy 126.3 119.25)))
+    (arrow1a (pts (xy 126.3 119.25) (xy 125.713579 118.123496)))
+    (arrow1b (pts (xy 126.3 119.25) (xy 126.886421 118.123496)))
+    (arrow2a (pts (xy 126.3 60.5) (xy 125.713579 61.626504)))
+    (arrow2b (pts (xy 126.3 60.5) (xy 126.886421 61.626504)))
+  )
+  (dimension 52.5 (width 0.15) (layer Dwgs.User)
+    (gr_text "52.500 mm" (at 99.25 56.8) (layer Dwgs.User)
+      (effects (font (size 1 1) (thickness 0.15)))
+    )
+    (feature1 (pts (xy 125.5 61.3) (xy 125.5 57.513579)))
+    (feature2 (pts (xy 73 61.3) (xy 73 57.513579)))
+    (crossbar (pts (xy 73 58.1) (xy 125.5 58.1)))
+    (arrow1a (pts (xy 125.5 58.1) (xy 124.373496 58.686421)))
+    (arrow1b (pts (xy 125.5 58.1) (xy 124.373496 57.513579)))
+    (arrow2a (pts (xy 73 58.1) (xy 74.126504 58.686421)))
+    (arrow2b (pts (xy 73 58.1) (xy 74.126504 57.513579)))
   )
   (gr_text 5V (at 75.25 95.25 90) (layer F.SilkS)
@@
   (segment (start 118.41 77.16) (end 118.41 79.25) (width 0.5) (layer F.Cu) (net 0))
   (segment (start 117 75.75) (end 118.41 77.16) (width 0.5) (layer F.Cu) (net 0))
-  (segment (start 123.51 101.49) (end 123.5 101.5) (width 2) (layer B.Cu) (net 0))
-  (segment (start 90.56 65.32) (end 90.56 66.69) (width 2) (layer B.Cu) (net 0))
-  (segment (start 113.38 79.25) (end 113.38 78.12) (width 2) (layer B.Cu) (net 0))
-  (segment (start 113.38 79.25) (end 113.38 80.62) (width 2) (layer B.Cu) (net 0))
-  (segment (start 113.38 89.75) (end 113.38 88.38) (width 2) (layer B.Cu) (net 0))
-  (segment (start 113.38 89.75) (end 113.38 91.38) (width 2) (layer B.Cu) (net 0))
-  (segment (start 123.51 97.5) (end 123.51 95.76) (width 2) (layer B.Cu) (net 0))
-  (segment (start 123.5 97.51) (end 123.51 97.5) (width 2) (layer B.Cu) (net 0))
-  (segment (start 123.5 101.5) (end 123.5 97.51) (width 2) (layer B.Cu) (net 0))
-  (segment (start 123.5 101.5) (end 123.5 103.5) (width 2) (layer B.Cu) (net 0))
-  (zone (net 0) (net_name "") (layer B.Cu) (hatch edge 0.508)
-    (connect_pads (clearance 0.508))
-    (min_thickness 0.254)
-    (fill yes (arc_segments 32) (thermal_gap 1) (thermal_bridge_width 1))
-    (polygon
-      (pts
-        (xy 125.5 119.25) (xy 73 119.25) (xy 73 60.5) (xy 125.5 60.5)
-      )
-    )
-  )
 )

Commit message: added bom
Routing:
- net (no net): track 564.2 -> 577.5 mm
- added copper zone on B.Cu, net (none)
